Commit message: add gripper2 and works

File: Tools/sitl_gazebo/models/gripper1/gripper1.urdf (robot description, URDF)
Before this commit: robot gripper2, 3 links, 2 joints
Links:
- link base_link: mass 0.11906 -> 0.18394; geometry collision mesh filename=package://gripper1/meshes/base_link.STL; visual mesh filename=package://gripper1/meshes/base_link.STL
- link left_link: mass 0.026471 -> 0.19697; geometry collision mesh filename=package://gripper1/meshes/left_link.STL; visual mesh filename=package://gripper1/meshes/left_link.STL
- link right_link: mass 0.027594 -> 0.098607; geometry collision mesh filename=package://gripper1/meshes/right_link.STL; visual mesh filename=package://gripper1/meshes/right_link.STL
Joints:
- joint left_joint: axis 0 -1 0 -> -1 0 0; limit lower=-3 upper=3 effort=1 velocity=1 -> lower=-0.05 upper=0.05 effort=1 velocity=0.1; origin xyz=-0.0135 0 0.01 rpy=0 0 0 -> xyz=-0.051103 -0.052 0.0005 rpy=0 0 0; type revolute -> prismatic
- joint right_joint: axis 0 -1 0 -> 1 0 0; limit lower=-3 upper=3 effort=1 velocity=1 -> lower=-0.05 upper=0.05 effort=1 velocity=0.1; origin xyz=-0.0135 0 -0.014 rpy=0 0 0 -> xyz=0.037773 -0.056 0.0005 rpy=3.1416 0 3.1416; type revolute -> prismatic
