Commit message: :bug: fix landing leg bug and work good

File: Tools/sitl_gazebo/models/landing_leg/landing_leg.urdf (robot description, URDF)
Before this commit: robot landing_leg, 9 links, 8 joints
Links:
- link base_link: mass 0.62479 -> 0.12479
- link link2_1: mass 0.01515 -> 0.0151495097581002
Joints:
- joint joint1: limit lower=0 upper=0 effort=0 velocity=0 -> lower=-3 upper=3 effort=10 velocity=10
- joint joint1_1: limit lower=0 upper=0 effort=0 velocity=0 -> lower=-5 upper=5 effort=10 velocity=10; origin xyz=-0.015 -0.12417 -0.19241 rpy=0 0 0 -> xyz=-0.015 -0.229 0 rpy=0 0 0
- joint joint2: limit lower=0 upper=0 effort=0 velocity=0 -> lower=-3 upper=3 effort=10 velocity=10
- joint joint2_1: limit lower=0 upper=0 effort=0 velocity=0 -> lower=-5 upper=5 effort=10 velocity=10; origin xyz=0.12417 -0.015 -0.19241 rpy=0 0 0 -> xyz=0.229 -0.015 0 rpy=0 0 0
- joint joint3: limit lower=0 upper=0 effort=0 velocity=0 -> lower=-3 upper=3 effort=10 velocity=10
- joint joint3_1: limit lower=0 upper=0 effort=0 velocity=0 -> lower=-5 upper=5 effort=10 velocity=10; origin xyz=0.015 0.12417 -0.19241 rpy=0 0 0 -> xyz=0.015 0.229 0 rpy=0 0 0
- joint joint4: limit lower=0 upper=0 effort=0 velocity=0 -> lower=-3 upper=3 effort=10 velocity=10
- joint joint4_1: limit lower=0 upper=0 effort=0 velocity=0 -> lower=-5 upper=5 effort=10 velocity=10; origin xyz=-0.12417 0.016 -0.19241 rpy=0 0 0 -> xyz=-0.229 0.016 0 rpy=0 0 0
